File: output/output.sch (KiCad schematic (older format))
At the start: 60 parts, among them J1 AudioJack2_SwitchT, J2 AudioJack2_SwitchT, J3 Conn_02x05_Odd_Even, J4 AudioJack3, J5 AudioJack3, Q1 MMBT3904, Q2 MMBT3904, U1 NE5532, U2 TL074, U3 NE5532

Commit message: Board layout for Output module
Parts:
- J1, J2: footprint footprints:Jack_3.5mm_QingPu_WQP-PJ398SM_Vertical_CircularHoles -> kicad_lib:Jack_3.5mm_QingPu_WQP-PJ398SM_Vertical_CircularHoles
- J4, J5: footprint footprints:Jack_3.5mm_QingPu_WQP-WQP419GR_Vertical_CircularHoles -> kicad_lib:Jack_3.5mm_QingPu_WQP-WQP419GR_Vertical_CircularHoles
- RV1, RV2: footprint footprints:Potentiometer_Song_Huei_R1214G_Dual_Vertical -> kicad_lib:Potentiometer_Song_Huei_R1214G_Dual_Vertical
Changed lines of the file:
@@
 F 0 "J2" H 2582 3675 50  0000 C CNN
 F 1 "AudioJack2_SwitchT" H 2150 3600 50  0001 C CNN
-F 2 "footprints:Jack_3.5mm_QingPu_WQP-PJ398SM_Vertical_CircularHoles" H 2550 3350 50  0001 C CNN
+F 2 "kicad_lib:Jack_3.5mm_QingPu_WQP-PJ398SM_Vertical_CircularHoles" H 2550 3350 50  0001 C CNN
 F 3 "~" H 2550 3350 50  0001 C CNN
 	1    2550 3350
@@
 F 0 "J4" H 8770 2583 50  0000 R CNN
 F 1 "AudioJack3" H 8770 2674 50  0000 R CNN
-F 2 "footprints:Jack_3.5mm_QingPu_WQP-WQP419GR_Vertical_CircularHoles" H 9050 2650 50  0001 C CNN
+F 2 "kicad_lib:Jack_3.5mm_QingPu_WQP-WQP419GR_Vertical_CircularHoles" H 9050 2650 50  0001 C CNN
 F 3 "~" H 9050 2650 50  0001 C CNN
 	1    9050 2650
@@
 F 0 "J5" H 8920 5183 50  0000 R CNN
 F 1 "AudioJack3" H 8920 5274 50  0000 R CNN
-F 2 "footprints:Jack_3.5mm_QingPu_WQP-WQP419GR_Vertical_CircularHoles" H 9200 5250 50  0001 C CNN
+F 2 "kicad_lib:Jack_3.5mm_QingPu_WQP-WQP419GR_Vertical_CircularHoles" H 9200 5250 50  0001 C CNN
 F 3 "~" H 9200 5250 50  0001 C CNN
 	1    9200 5250
@@
 F 0 "RV2" V 5500 5850 50  0000 R CNN
 F 1 "100k" V 5400 5900 50  0000 R CNN
-F 2 "footprints:Potentiometer_Song_Huei_R1214G_Dual_Vertical" H 5700 5525 50  0001 C CNN
+F 2 "kicad_lib:Potentiometer_Song_Huei_R1214G_Dual_Vertical" H 5700 5525 50  0001 C CNN
 F 3 "~" H 5700 5525 50  0001 C CNN
 	1    5450 5600
@@
 F 0 "RV1" V 5700 2900 50  0000 R CNN
 F 1 "100k" V 5600 2950 50  0000 R CNN
-F 2 "footprints:Potentiometer_Song_Huei_R1214G_Dual_Vertical" H 5900 2625 50  0001 C CNN
+F 2 "kicad_lib:Potentiometer_Song_Huei_R1214G_Dual_Vertical" H 5900 2625 50  0001 C CNN
 F 3 "~" H 5900 2625 50  0001 C CNN
 	1    5650 2700
@@
 F 0 "J1" H 2371 1829 50  0000 R CNN
 F 1 "AudioJack2_SwitchT" H 2582 2084 50  0001 C CNN
-F 2 "footprints:Jack_3.5mm_QingPu_WQP-PJ398SM_Vertical_CircularHoles" H 2550 1850 50  0001 C CNN
+F 2 "kicad_lib:Jack_3.5mm_QingPu_WQP-PJ398SM_Vertical_CircularHoles" H 2550 1850 50  0001 C CNN
 F 3 "~" H 2550 1850 50  0001 C CNN
 	1    2550 1850
