File: hex_wave_bank/pcb/hex_wave_bank.kicad_pcb (KiCad board)
At the start: 2 copper layers, 19 x 110 mm, 101 parts, among them J101 Conn_02x05_Odd_Even, J201 AudioJack2_SwitchT, J301 AudioJack2_SwitchT, J401 AudioJack2_SwitchT, J501 AudioJack2_SwitchT, J601 AudioJack2_SwitchT, J701 AudioJack2_SwitchT, U201 TL071HDBV, U301 TL071HDBV, U401 TL071HDBV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

Commit message: Redo grounds
Parts:
- moved C703 6.50 mm to (140.3, 130.5), turned to -90 degrees
- moved C303 6.50 mm to (140.3, 67.5), turned to -90 degrees
- moved C403 6.50 mm to (140.3, 83.2), turned to -90 degrees
- moved C503 6.50 mm to (140.3, 99.0), turned to -90 degrees
- moved C603 6.50 mm to (140.3, 114.8), turned to -90 degrees
- moved C203 6.50 mm to (140.3, 51.7), turned to -90 degrees
- moved C204 3.83 mm to (144.4, 46.7), turned to 0 degrees
- moved C304 3.83 mm to (144.4, 62.5), turned to 0 degrees
- moved C404 3.83 mm to (144.4, 78.2), turned to 0 degrees
- moved C504 3.83 mm to (144.4, 94.0), turned to 0 degrees
- moved C604 3.83 mm to (144.4, 109.8), turned to 0 degrees
- moved C704 3.83 mm to (144.4, 125.5), turned to 0 degrees
- moved R702 2.25 mm to (146.4, 137.6), turned to 90 degrees
- moved R302 2.25 mm to (146.4, 74.6), turned to 90 degrees
- moved R402 2.25 mm to (146.4, 90.3), turned to 90 degrees
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Routing:
- net GND: track 82.6 -> 69.7 mm, vias 12 -> 24
- net VEE: track 184.3 -> 171.8 mm
- net VCC: track 133.0 -> 140.9 mm
- net Net-(R303-Pad2): track 25.6 -> 28.6 mm
- net Net-(R603-Pad2): track 25.6 -> 28.6 mm
- net Net-(R703-Pad2): track 25.6 -> 28.6 mm
- net Net-(R403-Pad2): track 25.6 -> 28.6 mm
- net Net-(R503-Pad2): track 25.6 -> 28.6 mm
- net Net-(R203-Pad2): track 25.6 -> 28.6 mm
- net Net-(D601-K): track 8.88 -> 10.6 mm
- net Net-(D501-K): track 8.88 -> 10.6 mm
- net Net-(D701-K): track 8.88 -> 10.6 mm
- net Net-(D301-K): track 8.88 -> 10.6 mm
- net Net-(D201-K): track 8.88 -> 10.6 mm
- net Net-(D401-K): track 8.88 -> 10.6 mm
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Other:
- board text added: "Hex Wave Bank v1.1 www.birchavenue.org"
- board text removed: "Hex Wave Bank v1.0 www.birchavenue.org"
