File: hex_wave_bank/pcb/hex_wave_bank.kicad_sch (KiCad schematic)
At the start: 5 parts, among them J101 Conn_02x05_Odd_Even

Commit message: Add another ground plane, add capacitor values
Parts:
- C101, C102: value C_Polarized -> C_Polarized 10 uF
Changed lines of the file:
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@@
 			)
 		)
-		(property "Value" "C_Polarized"
+		(property "Value" "C_Polarized 10 uF"
 			(at 113.284 86.868 0)
 			(effects
@@
 			)
 		)
-		(property "Value" "C_Polarized"
+		(property "Value" "C_Polarized 10 uF"
 			(at 113.284 79.248 0)
 			(effects
@@
 		)
 		(instances
-			(project "fixed_sin_bank"
+			(project "hex_wave_bank"
 				(path "/fcaa2633-3922-4eef-aafe-407dcfc8954a"
 					(page "2")
@@
 		)
 		(instances
-			(project "fixed_sin_bank"
+			(project "hex_wave_bank"
 				(path "/fcaa2633-3922-4eef-aafe-407dcfc8954a"
 					(page "3")
@@
 		)
 		(instances
-			(project "fixed_sin_bank"
+			(project "hex_wave_bank"
 				(path "/fcaa2633-3922-4eef-aafe-407dcfc8954a"
 					(page "6")
@@
 		)
 		(instances
-			(project "fixed_sin_bank"
+			(project "hex_wave_bank"
 				(path "/fcaa2633-3922-4eef-aafe-407dcfc8954a"
 					(page "7")
@@
 		)
 		(instances
-			(project "fixed_sin_bank"
+			(project "hex_wave_bank"
 				(path "/fcaa2633-3922-4eef-aafe-407dcfc8954a"
 					(page "4")
@@
 		)
 		(instances
-			(project "fixed_sin_bank"
+			(project "hex_wave_bank"
 				(path "/fcaa2633-3922-4eef-aafe-407dcfc8954a"
 					(page "5")
